File: hackpad.kicad_sch (KiCad schematic)
At the start: 0 parts

Commit message: Add files via upload
Parts:
- added D1, D2: SK6812MINI, LED_SMD:LED_SK6812MINI_PLCC4_3.5x3.5mm_P1.75mm, symbol LED:SK6812MINI
- added SW1, SW2, SW3, SW4: SW_Push, HotSwap:Hotswap_MX_1.00u, symbol Switch:SW_Push
- added U1: XIAO-RP2040-DIP, OPL:XIAO-RP2040-DIP, symbol OPL:XIAO-RP2040-DIP
Connections:
- new net: D1.1 (DOUT), D2.3 (DIN)
- new net: D1.3 (DIN), U1.5 (GPIO6/SDA)
- new net: SW3.2, U1.10 (GPIO4/MISO)
- new net: SW4.2, U1.11 (GPIO3/MOSI)
- new net: SW1.2, U1.8 (GPIO1/RX)
- new net: SW2.2, U1.9 (GPIO2/SCK)
- new net +5V: D1.4 (VDD), D2.4 (VDD), U1.14 (VBUS)
- new net GND: D1.2 (VSS), D2.2 (VSS), SW1.1, SW2.1, SW3.1, SW4.1, U1.13 (GND)
